File: DuoDMXL_hardware/Duo Tri-state Buffer Shield/DuoTristateBuffer.brd (EAGLE design)
At the start: 55.2 x 33.2 mm, 20 parts, among them U1 MAX1674EUA+T

Commit message: Small modifications
Connections:
- net GND: now also BATT.1; no longer BATT.2
- net VIN: now also BATT.2; no longer BATT.1
Routing:
- net GND: track 224.1 -> 231.4 mm
- net VIN: track 12.5 -> 14.0 mm
Other:
- board text added: "WRONG"
Changed lines of the file:
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@@
 <?xml version="1.0" encoding="utf-8"?>
 <!DOCTYPE eagle SYSTEM "eagle.dtd">
-<eagle version="8.0.0">
+<eagle version="8.0.2">
 <drawing>
 <settings>
@@
 <text x="47.4" y="81.9" size="1.778" layer="22" rot="MR0">DUO Tri-state buffer v.1.0</text>
 <text x="41.8" y="79.4" size="1.778" layer="22" rot="MR0">Fabian Reyes</text>
+<text x="-15.2" y="69.3" size="1.778" layer="48">WRONG</text>
+<wire x1="-6.1" y1="72" x2="2.4" y2="72" width="0.4064" layer="48"/>
+<wire x1="2.4" y1="72" x2="2.4" y2="80.2" width="0.4064" layer="48"/>
 </plain>
 <attributes>
@@
 <element name="SV1" library="con-lsta" package="FE12" value="" x="22.86" y="92.71">
 <attribute name="MF" value="" x="22.86" y="92.71" size="1.778" layer="27" display="off"/>
-<attribute name="OC_NEWARK" value="unknown" x="22.86" y="92.71" size="1.778" layer="27" display="off"/>
 <attribute name="MPN" value="" x="22.86" y="92.71" size="1.778" layer="27" display="off"/>
 <attribute name="OC_FARNELL" value="unknown" x="22.86" y="92.71" size="1.778" layer="27" display="off"/>
+<attribute name="OC_NEWARK" value="unknown" x="22.86" y="92.71" size="1.778" layer="27" display="off"/>
 </element>
 <element name="SV2" library="con-lsta" package="FE12" value="" x="22.83" y="74.91">
 <attribute name="MF" value="" x="22.83" y="74.91" size="1.778" layer="27" display="off"/>
-<attribute name="OC_NEWARK" value="unknown" x="22.83" y="74.91" size="1.778" layer="27" display="off"/>
 <attribute name="MPN" value="" x="22.83" y="74.91" size="1.778" layer="27" display="off"/>
 <attribute name="OC_FARNELL" value="unknown" x="22.83" y="74.91" size="1.778" layer="27" display="off"/>
+<attribute name="OC_NEWARK" value="unknown" x="22.83" y="74.91" size="1.778" layer="27" display="off"/>
 </element>
 <element name="SV3" library="con-lsta" package="FE12" value="" x="22.86" y="95.45">
 <attribute name="MF" value="" x="22.86" y="95.45" size="1.778" layer="27" display="off"/>
-<attribute name="OC_NEWARK" value="unknown" x="22.86" y="95.45" size="1.778" layer="27" display="off"/>
 <attribute name="MPN" value="" x="22.86" y="95.45" size="1.778" layer="27" display="off"/>
 <attribute name="OC_FARNELL" value="unknown" x="22.86" y="95.45" size="1.778" layer="27" display="off"/>
+<attribute name="OC_NEWARK" value="unknown" x="22.86" y="95.45" size="1.778" layer="27" display="off"/>
 </element>
 <element name="SV4" library="con-lsta" package="FE12" value="" x="22.79" y="72.13">
 <attribute name="MF" value="" x="22.79" y="72.13" size="1.778" layer="27" display="off"/>
-<attribute name="OC_NEWARK" value="unknown" x="22.79" y="72.13" size="1.778" layer="27" display="off"/>
 <attribute name="MPN" value="" x="22.79" y="72.13" size="1.778" layer="27" display="off"/>
 <attribute name="OC_FARNELL" value="unknown" x="22.79" y="72.13" size="1.778" layer="27" display="off"/>
+<attribute name="OC_NEWARK" value="unknown" x="22.79" y="72.13" size="1.778" layer="27" display="off"/>
 </element>
 <element name="U1" library="Maxim" package="21-0036K" value="MAX1674EUA+T" x="20.54" y="86.81" rot="R180">
@@
 </element>
 <element name="SV5" library="con-lsta" package="FE12" value="" x="22.8" y="69.4">
+<attribute name="MF" value="" x="22.8" y="69.4" size="1.778" layer="27" display="off"/>
+<attribute name="MPN" value="" x="22.8" y="69.4" size="1.778" layer="27" display="off"/>
 <attribute name="OC_FARNELL" value="unknown" x="22.8" y="69.4" size="1.778" layer="27" display="off"/>
 <attribute name="OC_NEWARK" value="unknown" x="22.8" y="69.4" size="1.778" layer="27" display="off"/>
-<attribute name="MF" value="" x="22.8" y="69.4" size="1.778" layer="27" display="off"/>
-<attribute name="MPN" value="" x="22.8" y="69.4" size="1.778" layer="27" display="off"/>
 </element>
 </elements>
@@
 <wire x1="21.1" y1="86.4" x2="21.6244" y2="85.8" width="0.4064" layer="1"/>
 <wire x1="21.6244" y1="85.8" x2="22.7244" y2="85.8194" width="0.4064" layer="1"/>
-<contactref element="BATT" pad="2"/>
-<wire x1="4.8" y1="81.3" x2="7" y2="81.3" width="0.4064" layer="16"/>
-<wire x1="7" y1="81.3" x2="11.4" y2="76.7" width="0.4064" layer="16"/>
+<wire x1="7" y1="81.7" x2="11.4" y2="76.7" width="0.4064" layer="16"/>
 <wire x1="11.4" y1="76.7" x2="11.4" y2="74.91" width="0.4064" layer="16"/>
 <wire x1="27.79" y1="86.13" x2="31.35" y2="86.13" width="0.4064" layer="1"/>
@@
 <wire x1="49.21" y1="73.5" x2="52.31" y2="79.63" width="0.4064" layer="16"/>
 <contactref element="D1" pad="K"/>
-<wire x1="4.8" y1="84.43" x2="4.8" y2="81.3" width="0.4064" layer="16"/>
 <contactref element="SV5" pad="2"/>
 <wire x1="12.36" y1="67.7" x2="11.47" y2="68.5" width="0.4064" layer="16"/>
@@
 <wire x1="11.37" y1="69.4" x2="11.36" y2="69.4" width="0.4064" layer="16"/>
 <wire x1="11.36" y1="69.4" x2="11.36" y2="72.13" width="0.4064" layer="16"/>
+<contactref element="BATT" pad="1"/>
+<wire x1="4.8" y1="84.43" x2="7" y2="83.63" width="0.4064" layer="16"/>
+<wire x1="7" y1="82.8" x2="7" y2="83.63" width="0.4064" layer="16"/>
+<wire x1="7" y1="82.8" x2="7" y2="81.7" width="0.4064" layer="16"/>
+<wire x1="4.8" y1="79.3" x2="3" y2="80.4" width="0.4064" layer="16"/>
+<wire x1="3" y1="80.4" x2="3" y2="81.9" width="0.4064" layer="16"/>
+<wire x1="3" y1="81.9" x2="3.6" y2="82.8" width="0.4064" layer="16"/>
+<wire x1="3.6" y1="82.8" x2="7" y2="82.8" width="0.4064" layer="16"/>
 <wire x1="45.595" y1="88.3571" x2="45.7" y2="89.2" width="0" layer="19" extent="1-1"/>
 <wire x1="45.6" y1="79.5" x2="45.595" y2="78.8829" width="0" layer="19" extent="1-1"/>
@@
 <wire x1="8.86" y1="74.91" x2="8.82" y2="74.91" width="0.4064" layer="16"/>
 <wire x1="8.82" y1="72.13" x2="8.82" y2="74.91" width="0.4064" layer="16"/>
-<contactref element="BATT" pad="1"/>
-<wire x1="4.8" y1="79.3" x2="6.1" y2="79.3" width="0.4064" layer="16"/>
-<wire x1="6.1" y1="79.3" x2="8.86" y2="77" width="0.4064" layer="16"/>
-<wire x1="8.86" y1="77" x2="8.86" y2="74.91" width="0.4064" layer="16"/>
 <contactref element="SV5" pad="1"/>
 <wire x1="8.83" y1="69.4" x2="8.82" y2="69.4" width="0.4064" layer="16"/>
 <wire x1="8.82" y1="69.4" x2="8.82" y2="72.13" width="0.4064" layer="16"/>
+<contactref element="BATT" pad="2"/>
+<wire x1="4.8" y1="81.3" x2="5.6" y2="81.3" width="0.4064" layer="16"/>
+<wire x1="5.6" y1="81.3" x2="8.9" y2="77.7" width="0.4064" layer="16"/>
+<wire x1="8.9" y1="77.7" x2="8.86" y2="76.3" width="0.4064" layer="16"/>
+<wire x1="8.86" y1="76.3" x2="8.86" y2="74.91" width="0.4064" layer="16"/>
 </signal>
 <signal name="TX">
